File: eagle/analyzer/small_analyzer.brd (EAGLE design)
At the start: 91.4 x 34.3 mm, 36 parts, among them IC1 MCP604ST, IC2 TPS77301, IC3 TPS77350, U1 AD5933, U2 ATMEGA328P

Commit message: fixed drc laws
Parts:
- added S2: (no value), SparkFun-Electromechanical:TACTILE_SWITCH_SMD
- moved JP4 13.0 mm to (55.9, 3.81), turned to 0 degrees
- moved Y1 6.35 mm to (64.8, 8.89)
- moved LED2 5.08 mm to (69.8, 30.5)
- moved R15 5.08 mm to (69.8, 27.9)
- moved JP2 5.08 mm to (48.3, 30.5)
- moved C2 5.08 mm to (30.5, 5.08)
- moved C7 5.08 mm to (21.6, 7.62)
- moved C8 5.08 mm to (24.1, 7.62)
- moved IC1 5.08 mm to (12.7, 15.2)
- moved IC2 5.08 mm to (12.7, 24.1)
- moved R16 5.08 mm to (22.9, 12.7)
- moved R17 5.08 mm to (22.9, 17.8)
- moved C1 5.08 mm to (6.35, 20.3)
- moved R1 5.08 mm to (3.81, 19.1)
- moved R10 5.08 mm to (5.08, 24.1)
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Connections:
- new net N$16: S2.1, S2.2, U2.25
- net VCC: now also S2.3, S2.4
Routing:
- net N$16: track 0.00 -> 34.7 mm
- net +IN: track 73.6 -> 42.5 mm, vias 4 -> 2
- net VBAT: track 32.3 -> 48.5 mm
- net VIN: track 32.2 -> 47.3 mm
- net GND: track 247.0 -> 233.4 mm, vias 10 -> 0
- net N$5: track 8.94 -> 17.5 mm, vias 0 -> 2
- net IOUT2: track 31.0 -> 39.4 mm
- net MOSI: track 14.3 -> 21.0 mm, vias 1 -> 0
- net RST: track 34.8 -> 40.5 mm
- net VAMP: track 23.1 -> 17.5 mm, vias 4 -> 2
- net VCC: track 144.0 -> 139.4 mm, vias 8 -> 2
- net N$11: track 23.5 -> 19.1 mm, vias 2 -> 0
- net VREF: track 13.8 -> 10.1 mm
- net SCL: track 24.0 -> 27.0 mm, vias 2 -> 1
- net N$4: track 11.3 -> 14.2 mm, vias 0 -> 2
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Other:
- board size 91.4 x 34.3 mm -> 82.5 x 34.3 mm
- board text added: "Reset"
- board text added: "Sweep"
