File: eagle/analyzer/small_analyzer.sch (EAGLE design)
At the start: 39 parts, among them IC1 MCP604ST, IC2 TPS77301, IC3 TPS77350, U1 AD5933, U2 ATMEGA328P

Commit message: added dual voltage regulator to board
Parts:
- added IC4: (no value), AWJLEagleLib:LT3032
Other:
- note added: "LT3015"
Changed lines of the file:
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@@
 <?xml version="1.0" encoding="utf-8"?>
 <!DOCTYPE eagle SYSTEM "eagle.dtd">
-<eagle version="6.5.0">
+<eagle version="6.4">
 <drawing>
 <settings>
@@
 <part name="C9" library="SparkFun-Passives" deviceset="CAP" device="0603-CAP" value="0.1uF"/>
 <part name="GND2" library="SparkFun-Aesthetics" deviceset="GND" device=""/>
+<part name="IC4" library="AWJLEagleLib" deviceset="LT3032" device=""/>
 </parts>
 <sheets>
@@
 <text x="147.32" y="226.06" size="1.778" layer="91">ADR423_8MSOP</text>
 <text x="152.4" y="50.8" size="1.778" layer="91">AD8236_8MSOP</text>
+<text x="149.86" y="195.58" size="1.778" layer="91">LT3015</text>
 </plain>
 <instances>
@@
 <instance part="C9" gate="G$1" x="147.32" y="162.56"/>
 <instance part="GND2" gate="1" x="139.7" y="154.94"/>
+<instance part="IC4" gate="G$1" x="154.94" y="208.28"/>
 </instances>
 <busses>

Commit message: updated schematic to dual voltage regulator, errors in board
Parts:
- removed C2, C8: 0.1uF, SparkFun-Passives:CAP0603-CAP
- removed C7: 10uF, SparkFun-Passives:CAP0603-CAP
- removed IC3: TPS77350, texas:TPS77350
- added BAT+3V, BAT-3V: (no value), SparkFun-Electromechanical:BATTERY12MM
- added C10, C11, C12, C13: 10uF, SparkFun-Passives:CAP0603-CAP
- added C14, C15: 0.01uF, SparkFun-Passives:CAP0603-CAP
- added R1N, R1P, R2N, R2P: 100k, SparkFun-Passives:RESISTOR0805-RES
Connections:
- new net -VCC: C13.1, C15.1, IC4.ON, R2N.2
- new net N$13: BAT+3V.-, BAT-3V.+, C10.1, C11.2, IC4.GND
- new net N$14: BAT+3V.+, C11.1, IC4.!SP, IC4.IP
- new net N$18: C14.2, IC4.BP
- new net N$19: BAT-3V.-, C10.2, IC4.!SN, IC4.IN, IC4.IN@1
- new net N$20: C15.2, IC4.BN
- new net N$21: IC4.AJN, R1N.2, R2N.1
- new net N$22: IC4.AJP, R1P.1, R2P.2
- net GND: now also C12.2, C13.2, IC4.GND@1, R1N.1, R1P.2; no longer C2.2, C7.2, C8.2, IC3.GND
- net VBAT: no longer C7.1, C8.1, IC3.!RESET
- net VCC: now also C12.1, C14.1, IC4.OP, R2P.1; no longer C2.1, IC3.OUT@1
Other:
- note removed: "ADR423_8MSOP"
- moved on the sheet: IC1D, IC4, R16, R17

Commit message: analyzer version 1 as submitted for pcb fab
Parts:
- added C2, C7: 1u, SparkFun-Passives:CAP0603-CAP
- added JP6: M02PTH, SparkFun-Connectors:M02PTH
- BAT1: value (none) -> +3V
- BAT2: value (none) -> -3V
- renumbered BAT+3V to BAT1, BAT-3V to BAT2
Connections:
- net IOUT2 renamed IIN
- net VREF renamed VDC
- removed net +IN: IC1B.+IN, IC2.GND, JP3.3, R2.2, R5.1
- removed net -IN: IC2.FB\SENSE, JP3.4, R12.1
- removed net CS: U2.PB2(SS/OC1B)
- removed net N$14 (its old number): BAT1.+, C11.1, IC4.!SP, IC4.IP
- removed net N$17: U2.PC0(ADC0)
- new net +IOUT: C2.1, IC1B.+IN, JP3.3, R2.2, R5.1
- new net -IOUT: C7.2, JP3.4, R12.1
- new net A1: JP6.2, U2.PC1(ADC1)
- new net D6: JP6.1, U2.PD6(AIN0)
- new net N$24: C7.1, IC2.FB\SENSE
- new net N$25: C2.2, IC2.GND
- net VBAT: now also BAT1.+, C11.1, IC4.!SP, IC4.IP
Other:
- moved on the sheet: IC1D, JP3, R16, R17
